File: kicad/Esp32LoraBoard/Esp32LoraBoard.sch (KiCad schematic (older format))
At the start: 58 parts, among them J1 USB_B_Micro, J2 Power-Selector, J3 Testpoints, J4 ESP_PROG_JTAG, J5 Prog, J6 ext_Measure, J7 Measurement-Selector, J8 OLED_128x64, J9 Pin1-to-GND, Q1 UMH3N, Q2 Si2302DS_NMOS, Q3 Si2301DS_PMOS, Q4 Si2302DS_NMOS, Q5 Si2301DS_PMOS, Q6 Si2302DS_NMOS, SW1 Rotary_Encoder, SW2 Reset, U1 LM3940IMP-3.3, U2 ESP32-WROOM-32, U3 RFM95W-868S2

Commit message: Fixed: library path
Parts:
- AE1: symbol Device:Antenna_Shield -> Esp32LoraBoard-rescue:Antenna_Shield-Device
- BT1: symbol Device:Battery_Cell -> Esp32LoraBoard-rescue:Battery_Cell-Device
- C1, C10, C7, C8, C9: symbol Device:C -> Esp32LoraBoard-rescue:C-Device
- C2: symbol Device:CP_Small -> Esp32LoraBoard-rescue:CP_Small-Device
- C3, C4, C5, C6: symbol Device:C_Small -> Esp32LoraBoard-rescue:C_Small-Device
- FID1, FID2, FID3, FID4: symbol Mechanical:Fiducial -> Esp32LoraBoard-rescue:Fiducial-Mechanical
- J1: symbol Connector:USB_B_Micro -> Esp32LoraBoard-rescue:USB_B_Micro-Connector
- J2, J7: symbol Connector:Conn_01x03_Male -> Esp32LoraBoard-rescue:Conn_01x03_Male-Connector
- J3, J5: symbol Connector:Conn_01x05_Male -> Esp32LoraBoard-rescue:Conn_01x05_Male-Connector
- J4: symbol Connector_Generic:Conn_02x05_Odd_Even -> Esp32LoraBoard-rescue:Conn_02x05_Odd_Even-Connector_Generic
- J6: symbol Connector:Screw_Terminal_01x04 -> Esp32LoraBoard-rescue:Screw_Terminal_01x04-Connector
- J8: symbol Connector:Conn_01x04_Female -> Esp32LoraBoard-rescue:Conn_01x04_Female-Connector
- J9: symbol Connector:Conn_01x02_Male -> Esp32LoraBoard-rescue:Conn_01x02_Male-Connector
- Q2, Q4, Q6: symbol Device:Q_NMOS_GSD -> Esp32LoraBoard-rescue:Q_NMOS_GSD-Device
- Q3, Q5: symbol Device:Q_PMOS_GSD -> Esp32LoraBoard-rescue:Q_PMOS_GSD-Device
- R1, R10, R11, R12, R13, R14, R15, R2, R3, R4, R5, R6, R7, R8, R9: symbol Device:R -> Esp32LoraBoard-rescue:R-Device
- SW1: symbol Device:Rotary_Encoder_Switch -> Esp32LoraBoard-rescue:Rotary_Encoder_Switch-Device
- SW2: symbol Switch:SW_Push_Dual_x2 -> Esp32LoraBoard-rescue:SW_Push_Dual_x2-Switch
- TP1, TP2, TP3, TP4, TP5, TP6, TP7: symbol Connector:TestPoint -> Esp32LoraBoard-rescue:TestPoint-Connector
- U2: symbol RF_Module:ESP32-WROOM-32 -> Esp32LoraBoard-rescue:ESP32-WROOM-32-RF_Module
- U3: symbol RF_Module:RFM95W-868S2 -> Esp32LoraBoard-rescue:RFM95W-868S2-RF_Module
